Commit message: Added end effector and added plugins in gazebo

File: urdf/final_final_design_for_urdf.urdf (robot description, URDF)
Before this commit: robot final_final_design_for_urdf, 14 links, 13 joints
Links:
- removed link conecting_rod_end1_link
- removed link conecting_rod_end2_link
- removed link connecting_rod_coupler_link
- removed link end1_link
- removed link end2_link
- removed link lower_arm1_link
- removed link lower_arm2_link
- removed link push_rod_lower_arm_link
- removed link tringle1_link
- removed link tringle2_link
- removed link upper_arm_link
- added link end_effector_1_link, mass 0.0221251418758699; collision mesh filename=package://final_final_design_for_urdf/meshes/end_effector_1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; visual mesh filename=package://final_final_design_for_urdf/meshes/end_effector_1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
- added link end_effector_2_link, mass 0.000308029324600945; collision mesh filename=package://final_final_design_for_urdf/meshes/end_effector_2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; visual mesh filename=package://final_final_design_for_urdf/meshes/end_effector_2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
- added link end_effector_3_link, mass 0.0011129867228627; collision mesh filename=package://final_final_design_for_urdf/meshes/end_effector_3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; visual mesh filename=package://final_final_design_for_urdf/meshes/end_effector_3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
- added link end_effector_gripper_link, mass 0.000528572963966483; collision mesh filename=package://final_final_design_for_urdf/meshes/end_effector_g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; visual mesh filename=package://final_final_design_for_urdf/meshes/end_effector_g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
- added link end_effector_link, mass 0.0374839757136743; collision mesh filename=package://final_final_design_for_urdf/meshes/end_effector_l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; visual mesh filename=package://final_final_design_for_urdf/meshes/end_effector_l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
- added link end_effector_push_rod_link, mass 0.0374839757136743; collision mesh filename=package://final_final_design_for_urdf/meshes/end_effector_p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; visual mesh filename=package://final_final_design_for_urdf/meshes/end_effector_p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
- added link gripper_1_link, mass 0.0294248953782339; collision mesh filename=package://final_final_design_for_urdf/meshes/gripper_1_link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; visual mesh filename=package://final_final_design_for_urdf/meshes/gripper_1_link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
- added link gripper_2_link, mass 0.028834720369651; collision mesh filename=package://final_final_design_for_urdf/meshes/gripper_2_link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; visual mesh filename=package://final_final_design_for_urdf/meshes/gripper_2_link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
- added link gripper_link, mass 0.0294248953782339; collision mesh filename=package://final_final_design_for_urdf/meshes/gripper_link.S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; visual mesh filename=package://final_final_design_for_urdf/meshes/gripper_link.S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
- added link lower_arm_2_link, mass 0.219863068956833; collision mesh filename=package://final_final_design_for_urdf/meshes/lower_arm_2_li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; visual mesh filename=package://final_final_design_for_urdf/meshes/lower_arm_2_li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
- added link lower_arm_link, mass 0.219863068956833; collision mesh filename=package://final_final_design_for_urdf/meshes/lower_arm_link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; visual mesh filename=package://final_final_design_for_urdf/meshes/lower_arm_link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
- added link lower_arm_push_rod_coupler_link, mass 0.0324903102097775; collision mesh filename=package://final_final_design_for_urdf/meshes/lower_arm_push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; visual mesh filename=package://final_final_design_for_urdf/meshes/lower_arm_push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
- added link lower_arm_push_rod_link, mass 0.0123971170994329; collision mesh filename=package://final_final_design_for_urdf/meshes/lower_arm_push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; visual mesh filename=package://final_final_design_for_urdf/meshes/lower_arm_push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
- added link push_rod_end_effector_hip_link, mass 0.036107780403985; collision mesh filename=package://final_final_design_for_urdf/meshes/push_rod_end_e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; visual mesh filename=package://final_final_design_for_urdf/meshes/push_rod_end_e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
- added link push_rod_tringular_part_link, mass 0.00528822520415445; collision mesh filename=package://final_final_design_for_urdf/meshes/push_rod_tring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; visual mesh filename=package://final_final_design_for_urdf/meshes/push_rod_tring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
- added link tringular_part_lower_arm_link, mass 0.219863068956833; collision mesh filename=package://final_final_design_for_urdf/meshes/tringular_part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; visual mesh filename=package://final_final_design_for_urdf/meshes/tringular_part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
- added link tringular_push_rod_end_effector_link, mass 0.0251209380030328; collision mesh filename=package://final_final_design_for_urdf/meshes/tringular_push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; visual mesh filename=package://final_final_design_for_urdf/meshes/tringular_push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
- added link upper_link, mass 0.242573064725253; collision mesh filename=package://final_final_design_for_urdf/meshes/upper_link.STL; visual mesh filename=package://final_final_design_for_urdf/meshes/upper_link.STL
- link base_link: mass 0.418240339281201 -> 2.75370711603794; geometry collision mesh filename=package://final_final_design_for_urdf/meshes/base_link.STL; visual mesh filename=package://final_final_design_for_urdf/meshes/base_link.STL
- link hip_link: mass 0.407289435418519 -> 0.372958358086122; geometry collision mesh filename=package://final_final_design_for_urdf/meshes/hip_link.STL; visual mesh filename=package://final_final_design_for_urdf/meshes/hip_link.STL
Joints:
- removed joint conecting_rod_end1_joint
- removed joint conecting_rod_end2_joint
- removed joint connecting_rod_lower_arm1_joint
- removed joint end1_joint
- removed joint end2_link
- removed joint lower_arm1_joint
- removed joint lower_arm2_link
- removed joint push_rod_lower_arm_joint
- removed joint tringle1_joint
- removed joint tringle2_link
- removed joint upper_arm_link
- added joint end_effector_1_joint: type revolute, parent end_effector_link, child end_effector_1_link, origin xyz=0.008499 -0.021 0.04975 rpy=0 0 1.5524, axis 0 0 -1, limit lower=-3.14 upper=3.14 effort=1 velocity=0.01
- added joint end_effector_2_joint: type revolute, parent end_effector_1_link, child end_effector_2_link, origin xyz=-0.019875 2.5E-05 0.0246 rpy=-3.105 0 3.1416, axis -1 0 0, limit lower=-3.14 upper=3.14 effort=1 velocity=0.01
- added joint end_effector_3_joint: type revolute, parent end_effector_2_link, child end_effector_3_link, origin xyz=0.004475 0 0.01275 rpy=-1.8857 0 -3.1416, axis 1 0 0, limit lower=-3.14 upper=3.14 effort=1 velocity=0.01
- added joint end_effector_gripper_joint: type revolute, parent end_effector_3_link, child end_effector_gripper_link, origin xyz=0.01 0 0.045 rpy=-2.1377 0 0, axis 1 0 0, limit lower=-3.14 upper=3.14 effort=1 velocity=0.01
- added joint end_effector_joint: type revolute, parent lower_arm_link, child end_effector_link, origin xyz=-0.00040599 0 0.25 rpy=-0.79007 0 3.1416, axis 1 0 0, limit lower=-3.14 upper=3.14 effort=1 velocity=0.01
- added joint end_effector_push_rod_joint: type revolute, parent tringular_push_rod_end_effector_link, child end_effector_push_rod_link, origin xyz=-0.0095 0 0.25 rpy=-0.79007 0 0, axis 1 0 0, limit lower=-3.14 upper=3.14 effort=1 velocity=0.01
- added joint gripper_1_joint: type revolute, parent end_effector_1_link, child gripper_1_link, origin xyz=-0.007 -0.014875 0.0486 rpy=0 0 0, axis -1 0 0, limit lower=-3.14 upper=3.14 effort=1 velocity=0.01
- added joint gripper_2_joint: type revolute, parent end_effector_1_link, child gripper_2_link, origin xyz=-0.007 0.014925 0.0486 rpy=0 0 0, axis 1 0 0, limit lower=-3.14 upper=3.14 effort=1 velocity=0.01
- added joint gripper_joint: type revolute, parent end_effector_gripper_link, child gripper_link, origin xyz=0 0 0 rpy=0 0 1, axis 0 0 1, limit lower=-3.14 upper=3.14 effort=1 velocity=0.01
- added joint lower_arm_2_joint: type revolute, parent lower_arm_push_rod_link, child lower_arm_2_link, origin xyz=0 0 0.25 rpy=1.7248 0 3.1416, axis -1 0 0, limit lower=-3.14 upper=3.14 effort=1 velocity=0.01
- added joint lower_arm_joint: type revolute, parent upper_link, child lower_arm_link, origin xyz=0.003905 0 0.25 rpy=-1.7248 0 0, axis 1 0 0, limit lower=-3.14 upper=3.14 effort=1 velocity=0.01
- added joint lower_arm_push_rod_coupler_joint: type revolute, parent hip_link, child lower_arm_push_rod_coupler_link, origin xyz=0 0 0.05 rpy=0.79879 0 -1.5708, axis 1 0 0, limit lower=-3.14 upper=3.14 effort=1 velocity=0.01
- added joint lower_arm_push_rod_joint: type revolute, parent lower_arm_push_rod_coupler_link, child lower_arm_push_rod_link, origin xyz=-0.005 0.0010839 0.05999 rpy=-1.4349 0 0, axis 1 0 0, limit lower=-3.14 upper=3.14 effort=1 velocity=0.01
- added joint push_rod_end_effector_hip_joint: type revolute, parent hip_link, child push_rod_end_effector_hip_link, origin xyz=-0.034641 0.034001 0.07 rpy=-0.6361 0 -1.5708, axis -1 0 0, limit lower=-3.14 upper=3.14 effort=1 velocity=0.01
- added joint push_rod_tringular_part_joint: type revolute, parent push_rod_end_effector_hip_link, child push_rod_tringular_part_link, origin xyz=0.005002 0 0.25 rpy=-0.9347 0 0, axis 1 0 0, limit lower=-3.14 upper=3.14 effort=1 velocity=0.01
- added joint tringular_part_lower_arm_joint: type revolute, parent push_rod_tringular_part_link, child tringular_part_lower_arm_link, origin xyz=0.032904 0.02 0.034641 rpy=-0.79007 0 0, axis 1 0 0, limit lower=-3.14 upper=3.14 effort=1 velocity=0.01
- added joint tringular_push_rod_end_effector_joint: type revolute, parent push_rod_tringular_part_link, child tringular_push_rod_end_effector_link, origin xyz=0 0 0.069282 rpy=0.79007 0 -3.1416, axis -1 0 0, limit lower=-3.14 upper=3.14 effort=1 velocity=0.01
- added joint upper_joint: type revolute, parent hip_link, child upper_link, origin xyz=0 0 0.05 rpy=-0.6361 0 -1.5708, axis 1 0 0, limit lower=-3.14 upper=3.14 effort=1 velocity=0.01
- joint hip_joint: axis 0 0 -1 -> 0 0 1; limit lower=0 upper=0 effort=0 velocity=0 -> lower=-3.14 upper=3.14 effort=1 velocity=0.01; origin xyz=0 0 0.0365 rpy=0 0 0 -> xyz=0 0 0.032703 rpy=0 0 0
